Commit message: Top camera calibration

File: ros2_ws/src/so101_description/urdf/so101_arm_macro.xacro (robot description, xacro)
@@ -6,5 +6,5 @@
 -->
 <robot xmlns:xacro="http://www.ros.org/wiki/xacro">
-  <xacro:macro name="so101_arm" params="prefix parent mount_xyz mount_rpy">
+  <xacro:macro name="so101_arm" params="prefix parent mount_xyz mount_rpy use_wrist_camera_mount:=false">
     <joint name="${prefix}arm_mount_joint" type="fixed">
       <origin xyz="${mount_xyz}" rpy="${mount_rpy}"/>
@@ -269,9 +269,17 @@
       </geometry>
     </collision>
-    <!-- Part wrist_roll_follower_so101_v1 -->
+    <!--
+      The integrated 32x32 UVC camera mount is a complete Wrist Roll
+      replacement, not an add-on. Its official STL is authored in millimetres.
+    -->
     <visual>
       <origin xyz="8.32667e-17 -0.000218214 0.000949706" rpy="-3.14159 -5.55112e-17 0"/>
       <geometry>
-        <mesh filename="package://so101_description/meshes/wrist_roll_follower_so101_v1.stl"/>
+        <xacro:if value="${use_wrist_camera_mount}">
+          <mesh filename="package://so101_description/meshes/wrist_cam_mount_32x32_uvc_module_so101.stl" scale="0.001 0.001 0.001"/>
+        </xacro:if>
+        <xacro:unless value="${use_wrist_camera_mount}">
+          <mesh filename="package://so101_description/meshes/wrist_roll_follower_so101_v1.stl"/>
+        </xacro:unless>
       </geometry>
       <material name="3d_printed"/>
@@ -280,5 +288,10 @@
       <origin xyz="8.32667e-17 -0.000218214 0.000949706" rpy="-3.14159 -5.55112e-17 0"/>
       <geometry>
-        <mesh filename="package://so101_description/meshes/wrist_roll_follower_so101_v1.stl"/>
+        <xacro:if value="${use_wrist_camera_mount}">
+          <mesh filename="package://so101_description/meshes/wrist_cam_mount_32x32_uvc_module_so101.stl" scale="0.001 0.001 0.001"/>
+        </xacro:if>
+        <xacro:unless value="${use_wrist_camera_mount}">
+          <mesh filename="package://so101_description/meshes/wrist_roll_follower_so101_v1.stl"/>
+        </xacro:unless>
       </geometry>
     </collision>
@@ -291,4 +304,30 @@
     <child link="${prefix}gripper_frame_link"/>
   </joint>
+  <!--
+    Center of the 27x27 mm four-M2-hole pattern for the optional 32x32 UVC
+    camera module. The frame origin is the camera mounting plate mid-plane,
+    not the gripper TCP or the camera optical center. The CAD mesh origin,
+    millimetre scale, and visual Rx(pi) transform are already included here.
+    +Z is normal to the mounting plate.
+  -->
+  <xacro:if value="${use_wrist_camera_mount}">
+    <link name="${prefix}wrist_camera_mount_center_link"/>
+    <joint name="${prefix}wrist_camera_mount_center_joint" type="fixed">
+      <origin xyz="0.00250008 -0.07292374 0.00595299" rpy="-2.70526034 0 0"/>
+      <parent link="${prefix}gripper_link"/>
+      <child link="${prefix}wrist_camera_mount_center_link"/>
+    </joint>
+    <!--
+      Center of the temporary rigid yellow registration marker on the outer
+      surface of the 4 mm printed mounting plate. The visible surface is
+      local -Z from the CAD mid-plane; paper thickness is neglected.
+    -->
+    <link name="${prefix}wrist_registration_marker_link"/>
+    <joint name="${prefix}wrist_registration_marker_joint" type="fixed">
+      <origin xyz="0 0 -0.002" rpy="0 0 0"/>
+      <parent link="${prefix}wrist_camera_mount_center_link"/>
+      <child link="${prefix}wrist_registration_marker_link"/>
+    </joint>
+  </xacro:if>
   <!-- Link moving_jaw_so101_v1 -->
   <link name="${prefix}moving_jaw_link">
@@ -324,34 +363,53 @@
   <!-- Joint from wrist to gripper -->
   <joint name="${prefix}wrist_roll_joint" type="revolute">
-    <origin xyz="5.55112e-17 -0.0611 0.0181" rpy="1.5708 0.0486795 3.14159"/>
+    <!--
+      2026-07-26 left-arm physical Home: upstream q=-90deg is the new q=0.
+      The joint origin absorbs that rotation so raw 2048, ROS q=0, MoveIt
+      Home, and Isaac q=0 retain one shared meaning.
+    -->
+    <origin xyz="5.55112e-17 -0.0611 0.0181" rpy="1.57087172410138 -1.52211682665642 3.14151451327097"/>
     <parent link="${prefix}wrist_link"/>
     <child link="${prefix}gripper_link"/>
-    <axis xyz="0 0 -1"/>
-    <limit effort="10" velocity="10" lower="-2.84121" upper="2.74385"/>
+    <!--
+      2026-07-29 external rigid-target metrology: positive ROS feedback
+      rotates this physical joint about local +Z.
+    -->
+    <axis xyz="0 0 1"/>
+    <limit effort="10" velocity="10" lower="-4.3146463267949" upper="1.2704136732051"/>
   </joint>
   <!-- Joint from lower_arm to wrist -->
   <joint name="${prefix}wrist_flex_joint" type="revolute">
-    <origin xyz="-0.1349 0.0052 3.62355e-17" rpy="4.02456e-15 8.67362e-16 -1.5708"/>
+    <!--
+      Upstream q=-64.898281239deg is the new q=0. The 2026-07-30
+      eye-to-hand external metrology refined the visual -57.5deg baseline by
+      -7.398281239deg. Hardware raw 2048 and ROS feedback zero are unchanged.
+    -->
+    <origin xyz="-0.1349 0.0052 3.62355e-17" rpy="2.88657986402541e-15 -2.88657986402541e-15 -0.438111313497813"/>
     <parent link="${prefix}lower_arm_link"/>
     <child link="${prefix}wrist_link"/>
     <axis xyz="0 0 -1"/>
-    <limit effort="10" velocity="10" lower="-1.65806" upper="1.65806"/>
+    <limit effort="10" velocity="10" lower="-0.525371313497813" upper="2.790748686502188"/>
   </joint>
   <!-- Joint from upper_arm to lower_arm -->
-  <!-- Note: 5-degree calibration offset applied to joint limits -->
   <joint name="${prefix}elbow_joint" type="revolute">
-    <origin xyz="-0.11257 -0.028 1.73763e-16" rpy="-3.63608e-16 8.74301e-16 1.5708"/>
+    <!-- Upstream q=-55deg is the new q=0. -->
+    <origin xyz="-0.11257 -0.028 1.73763e-16" rpy="6.66133814775094e-16 8.88178419700125e-16 2.53073108859688"/>
     <parent link="${prefix}upper_arm_link"/>
     <child link="${prefix}lower_arm_link"/>
     <axis xyz="0 0 -1"/>
-    <limit effort="10" velocity="10" lower="-1.69" upper="1.69"/>
+    <limit effort="10" velocity="10" lower="-0.730068911403119" upper="2.64993108859688"/>
   </joint>
   <!-- Joint from shoulder to upper_arm -->
   <joint name="${prefix}shoulder_joint" type="revolute">
-    <origin xyz="-0.0303992 -0.0182778 -0.0542" rpy="-1.5708 -1.5708 0"/>
+    <!-- Upstream q=+90deg is the new q=0. -->
+    <origin xyz="-0.0303992 -0.0182778 -0.0542" rpy="1.5707963267814 3.67320510319402e-06 3.14158898038469"/>
     <parent link="${prefix}shoulder_link"/>
     <child link="${prefix}upper_arm_link"/>
-    <axis xyz="0 0 -1"/>
-    <limit effort="10" velocity="10" lower="-1.74533" upper="1.74533"/>
+    <!--
+      2026-07-29 external rigid-target metrology: positive ROS feedback
+      rotates this physical joint about local +Z.
+    -->
+    <axis xyz="0 0 1"/>
+    <limit effort="10" velocity="10" lower="-0.174533673205103" upper="3.3161263267949"/>
   </joint>
   <!-- Joint from base to shoulder -->
@@ -360,5 +418,9 @@
     <parent link="${prefix}base_link"/>
     <child link="${prefix}shoulder_link"/>
-    <axis xyz="0 0 -1"/>
+    <!--
+      2026-07-29 external rigid-target metrology: positive ROS feedback
+      rotates this physical joint about local +Z.
+    -->
+    <axis xyz="0 0 1"/>
     <limit effort="10" velocity="10" lower="-1.91986" upper="1.91986"/>
   </joint>

File: ros2_ws/src/so101_description/urdf/so101_left.urdf.xacro (robot description, xacro)
@@ -5,6 +5,11 @@
   <xacro:arg name="mount_rpy" default="0 0 0"/>
   <xacro:arg name="use_mock_hardware" default="false"/>
+  <xacro:arg name="use_wrist_camera_mount" default="true"/>
+  <xacro:arg name="use_overhead_webcam_mount" default="false"/>
+  <xacro:arg name="top_camera_xyz" default="0 0.2344404 0"/>
+  <xacro:arg name="top_camera_optical_rpy" default="1.5707963267948966 0 0"/>
   <xacro:include filename="so101_arm_macro.xacro"/>
   <xacro:include filename="so101_ros2_control.xacro"/>
+  <xacro:include filename="so101_overhead_webcam_mount.xacro"/>
   <material name="3d_printed">
     <color rgba="1.0 0.82 0.12 1.0"/>
@@ -14,4 +19,12 @@
   </material>
   <link name="workcell_base_link"/>
+  <xacro:if value="$(arg use_overhead_webcam_mount)">
+    <xacro:so101_overhead_webcam_mount
+      prefix="top_"
+      parent="workcell_base_link"
+      camera_xyz="$(arg top_camera_xyz)"
+      camera_optical_rpy="$(arg top_camera_optical_rpy)"
+    />
+  </xacro:if>
   <xacro:so101_arm
     prefix="$(arg arm_slot)_"
@@ -19,4 +32,5 @@
     mount_xyz="$(arg mount_xyz)"
     mount_rpy="$(arg mount_rpy)"
+    use_wrist_camera_mount="$(arg use_wrist_camera_mount)"
   />
   <xacro:if value="$(arg use_mock_hardware)">

Commit message: dual-arm-integration

File: ros2_ws/src/so101_description/urdf/so101_arm_macro.xacro (robot description, xacro)
@@ -6,5 +6,12 @@
 -->
 <robot xmlns:xacro="http://www.ros.org/wiki/xacro">
-  <xacro:macro name="so101_arm" params="prefix parent mount_xyz mount_rpy use_wrist_camera_mount:=false">
+  <xacro:macro name="so101_arm" params="
+    prefix parent mount_xyz mount_rpy use_wrist_camera_mount:=false
+    base_lower:=-1.91986 base_upper:=1.91986
+    shoulder_lower:=-0.174533673205103 shoulder_upper:=3.3161263267949
+    elbow_lower:=-0.730068911403119 elbow_upper:=2.64993108859688
+    wrist_flex_lower:=-0.525371313497813 wrist_flex_upper:=2.790748686502188
+    wrist_roll_lower:=-4.3146463267949 wrist_roll_upper:=1.2704136732051
+  ">
     <joint name="${prefix}arm_mount_joint" type="fixed">
       <origin xyz="${mount_xyz}" rpy="${mount_rpy}"/>
@@ -376,5 +383,5 @@
     -->
     <axis xyz="0 0 1"/>
-    <limit effort="10" velocity="10" lower="-4.3146463267949" upper="1.2704136732051"/>
+    <limit effort="10" velocity="10" lower="${wrist_roll_lower}" upper="${wrist_roll_upper}"/>
   </joint>
   <!-- Joint from lower_arm to wrist -->
@@ -389,5 +396,5 @@
     <child link="${prefix}wrist_link"/>
     <axis xyz="0 0 -1"/>
-    <limit effort="10" velocity="10" lower="-0.525371313497813" upper="2.790748686502188"/>
+    <limit effort="10" velocity="10" lower="${wrist_flex_lower}" upper="${wrist_flex_upper}"/>
   </joint>
   <!-- Joint from upper_arm to lower_arm -->
@@ -398,5 +405,5 @@
     <child link="${prefix}lower_arm_link"/>
     <axis xyz="0 0 -1"/>
-    <limit effort="10" velocity="10" lower="-0.730068911403119" upper="2.64993108859688"/>
+    <limit effort="10" velocity="10" lower="${elbow_lower}" upper="${elbow_upper}"/>
   </joint>
   <!-- Joint from shoulder to upper_arm -->
@@ -411,5 +418,5 @@
     -->
     <axis xyz="0 0 1"/>
-    <limit effort="10" velocity="10" lower="-0.174533673205103" upper="3.3161263267949"/>
+    <limit effort="10" velocity="10" lower="${shoulder_lower}" upper="${shoulder_upper}"/>
   </joint>
   <!-- Joint from base to shoulder -->
@@ -423,5 +430,5 @@
     -->
     <axis xyz="0 0 1"/>
-    <limit effort="10" velocity="10" lower="-1.91986" upper="1.91986"/>
+    <limit effort="10" velocity="10" lower="${base_lower}" upper="${base_upper}"/>
   </joint>
   </xacro:macro>

File: ros2_ws/src/so101_description/urdf/so101_overhead_webcam_mount.xacro (robot description, xacro)
@@ -11,10 +11,10 @@
 <robot xmlns:xacro="http://www.ros.org/wiki/xacro">
   <xacro:macro
-    name="so101_overhead_webcam_mount"
-    params="prefix parent camera_xyz:='0 0.2344404 0' camera_optical_rpy:='1.5707963267948966 0 0'">
+    name="so101_overhead_webcam_arm_base"
+    params="prefix parent mount_xyz:='0 0 0' mount_rpy:='0 0 0'">
     <xacro:property name="half_pi" value="1.5707963267948966"/>
     <!--
       The plate is aligned to the SO-101 base footprint grooves, not merely
-      centered on workcell_base_link. After the user-confirmed 180-degree
+      centered on its parent frame. After the user-confirmed 180-degree
       correction, raw STL axes map as (x,y,z)->(x,-z,y).
     -->
@@ -37,14 +37,18 @@
     </link>
     <joint name="${prefix}arm_base_joint" type="fixed">
-      <origin xyz="0 0 0" rpy="0 0 0"/>
+      <origin xyz="${mount_xyz}" rpy="${mount_rpy}"/>
       <parent link="${parent}"/>
       <child link="${prefix}arm_base_link"/>
     </joint>
+  </xacro:macro>
+  <xacro:macro
+    name="so101_overhead_webcam_tower"
+    params="prefix parent camera_xyz:='0 0.2344404 0' camera_optical_rpy:='1.5707963267948966 0 0'">
+    <xacro:property name="half_pi" value="1.5707963267948966"/>
     <!--
       User-confirmed side insertion: rotate the complete bottom+top assembly
-      180 degrees, then place its 37.4 mm edge in the left region seen from the
-      arm_base physical right side. The exact arm raw interval
-      x=-93.9209137..-56.5209137 mm matches the bottom raw x=0..37.4 mm edge.
-      Both floor bottoms remain at z=-5 mm.
+      180 degrees, then place its 37.4 mm edge in the arm-base groove. The
+      exact base raw interval x=-93.9209137..-56.5209137 mm matches the
+      bottom raw x=0..37.4 mm edge. Both floor bottoms remain at z=-5 mm.
     -->
     <link name="${prefix}cam_mount_bottom_link">
@@ -67,5 +71,5 @@
     <joint name="${prefix}cam_mount_bottom_joint" type="fixed">
       <origin xyz="0.0137353073 -0.1525445687 -0.005" rpy="${half_pi} 0 3.141592653589793"/>
-      <parent link="${prefix}arm_base_link"/>
+      <parent link="${parent}"/>
       <child link="${prefix}cam_mount_bottom_link"/>
     </joint>
@@ -111,3 +115,17 @@
     </joint>
   </xacro:macro>
+  <xacro:macro
+    name="so101_overhead_webcam_mount"
+    params="prefix parent camera_xyz:='0 0.2344404 0' camera_optical_rpy:='1.5707963267948966 0 0'">
+    <xacro:so101_overhead_webcam_arm_base
+      prefix="${prefix}"
+      parent="${parent}"
+    />
+    <xacro:so101_overhead_webcam_tower
+      prefix="${prefix}"
+      parent="${prefix}arm_base_link"
+      camera_xyz="${camera_xyz}"
+      camera_optical_rpy="${camera_optical_rpy}"
+    />
+  </xacro:macro>
 </robot>
