Commit message: feat(calibration): validate right-arm registration and clear pose

File: ros2_ws/src/so101_description/urdf/so101_overhead_webcam_mount.xacro (robot description, xacro)
@@ -30,7 +30,9 @@
       </visual>
       <collision>
-        <origin xyz="0.0211353034 0 -0.0014" rpy="0 0 0"/>
+        <origin xyz="0.0702562210 -0.0534304657 0" rpy="${half_pi} 0 0"/>
         <geometry>
-          <box size="0.08959999 0.15903915 0.0072"/>
+          <mesh
+            filename="package://so101_description/meshes/overhead_webcam_arm_base.stl"
+            scale="0.001 0.001 0.001"/>
         </geometry>
       </collision>
@@ -63,7 +65,9 @@
       </visual>
       <collision>
-        <origin xyz="0.0187 0.115475 0.0365125" rpy="0 0 0"/>
+        <origin xyz="0 0 0" rpy="0 0 0"/>
         <geometry>
-          <box size="0.0374 0.23095 0.093025"/>
+          <mesh
+            filename="package://so101_description/meshes/overhead_webcam_cam_mount_bottom.stl"
+            scale="0.001 0.001 0.001"/>
         </geometry>
       </collision>
@@ -90,7 +94,9 @@
       </visual>
       <collision>
-        <origin xyz="0 0.1172202 0" rpy="0 0 0"/>
+        <origin xyz="0 0 0" rpy="0 0 0"/>
         <geometry>
-          <box size="0.0254 0.2344404 0.036625"/>
+          <mesh
+            filename="package://so101_description/meshes/overhead_webcam_cam_mount_top_hinge_removed.stl"
+            scale="0.001 0.001 0.001"/>
         </geometry>
       </collision>
